Commit message: edit readme, and add spawn demo launch

File: marine_duckiebot_description/urdf/mybot.xacro (robot description, xacro)
@@ -4,9 +4,8 @@
   <xacro:property name="cameraMass" value="0.0001"/>
   <xacro:arg name="veh" default="$(arg veh)"/>
-  <xacro:include filename="$(find duckiebot_description)/urdf/wheel.urdf.xacro" />
-  <xacro:include filename="$(find duckiebot_description)/urdf/mybot.gazebo" />
-  <xacro:include filename="$(find duckiebot_description)/urdf/material.xacro" />
-  <xacro:include filename="$(find duckiebot_description)/urdf/plugin/usv_gazebo_dynamics_plugin_duckiebot.xacro" />
- <xacro:include filename="$(find velodyne_description)/urdf/example.urdf.xacro"/>
+  <xacro:include filename="$(find marine_duckiebot_description)/urdf/wheel.urdf.xacro" />
+  <xacro:include filename="$(find marine_duckiebot_description)/urdf/mybot.gazebo" />
+  <xacro:include filename="$(find marine_duckiebot_description)/urdf/material.xacro" />
+  <xacro:include filename="$(find marine_duckiebot_description)/urdf/plugin/usv_gazebo_dynamics_plugin_duckiebot.xacro" />
   <!-- Defines the macro for simulated GPS -->
   <xacro:include filename="$(find kingfisher_gazebo)/urdf/gps_gazebo.xacro" />
@@ -45,5 +44,5 @@
     <pose>0 0 0.0 0 0 0</pose>
     <inertial>
-      <mass value="15.0"/>
+      <mass value="35.0"/>
       <origin xyz="0.0 0 0.0" rpy=" 0 0 0"/>
       <inertia
@@ -144,5 +143,5 @@
     </collision>
     <visual>
-      <origin xyz="0.1 0 0.08" rpy="0 0.0 0.00"/>
+      <origin xyz="0.05 0 0.08" rpy="0 0.0 0.00"/>
       <geometry>
         <mesh filename="package://duckiebot_description/urdf/duck/dduck.dae" />
@@ -196,3 +195,7 @@
     <child link="camera"/>
   </joint>
+  <xacro:include filename="$(find velodyne_description)/urdf/VLP-16.urdf.xacro"/>
+  <VLP-16 parent="base_link" name="velodyne" topic="/velodyne_points" hz="10" samples="440">
+    <origin xyz="0 0 0.05" rpy="0 0 0" />
+  </VLP-16>
 </robot>

Commit message: fix path

File: marine_duckiebot_description/urdf/mybot.xacro (robot description, xacro)
@@ -118,5 +118,5 @@
       <origin xyz="-0.1 0 -0.05" rpy="0 0.0 1.57"/>
       <geometry>
-        <mesh filename="package://duckiebot_description/urdf/brian_base.stl" />
+        <mesh filename="package://marine_duckiebot_description/urdf/brian_base.stl" />
       </geometry>
       <!--material name="green"/-->
@@ -145,5 +145,5 @@
       <origin xyz="0.05 0 0.08" rpy="0 0.0 0.00"/>
       <geometry>
-        <mesh filename="package://duckiebot_description/urdf/duck/dduck.dae" />
+        <mesh filename="package://marine_duckiebot_description/urdf/duck/dduck.dae" />
       </geometry>
       <!--material name="green"/-->

Commit message: for global frame

File: marine_duckiebot_description/urdf/mybot.xacro (robot description, xacro)
@@ -156,5 +156,5 @@
     </inertial>
   </link>
-  <joint name="weight_joint" type="continuous">
+  <joint name="weight_joint" type="fixed">
     <axis xyz="0 0 0" />
     <origin xyz="-0.2 0 0.0" rpy="0 0.0 0"/>
